File: Hardware/STM32G0B1.kicad_sch (KiCad schematic)
At the start: 0 parts

Commit message: Finished the STM sheet mostly
- Added a bus for the STM32, as well as the individual peripherals
- Added LEDs for the Heartbeat and Fault outputs.
- Added 5 pushbuttons for the 5 channels, along with button debouncing
	- Refer to TI's button debouncing AN. RC low pass w/ 10ms time
	  constant. UNSURE if the schematic is correct, someone will
	  have to check.
Parts:
- added C1, C2, C3, C4, C5: 1u, symbol Device:C_Small_US
- added LED1, LED2: LED_Small, symbol Device:LED_Small
- added MCU1: STM32G0B1KETx, Package_QFP:LQFP-32_7x7mm_P0.8mm, symbol MCU_ST_STM32G0:STM32G0B1KETx
- added R1, R2, R3, R4, R5: 10k, symbol Device:R_Small_US
- added R6, R7: 1k, symbol Device:R_Small_US
- added SW1, SW2, SW3, SW4, SW5: SW_Push, symbol Switch:SW_Push
Connections:
- new net: R3.2, SW3.1
- new net: LED1.2 (A), R6.2
- new net: R1.2, SW1.1
- new net: R4.2, SW4.1
- new net: LED2.2 (A), R7.2
- new net: R5.2, SW5.1
- new net: R2.2, SW2.1
- new net 3v3: C1.1, C2.1, C3.1, C4.1, C5.1, MCU1.4 (VDD), SW1.2, SW2.2, SW3.2, SW4.2, SW5.2
- new net CAN1_RX: MCU1.22 (PA9/PA11)
- new net CAN1_TX: MCU1.23 (PA10/PA12)
- new net CAN_ADDR0: MCU1.18 (PA8)
- new net CAN_ADDR1: MCU1.19 (PA9/UCPD1_DBCC1)
- new net CAN_ADDR2: MCU1.21 (PA10/UCPD1_DBCC2)
- new net FAULT: MCU1.14 (PA7), R7.1
- new net GND: LED1.1 (K), LED2.1 (K), MCU1.5 (VSS)
- new net GPIO0: MCU1.8 (PA1)
- new net GPIO1: MCU1.9 (PA2)
- new net GPIO2: MCU1.10 (PA3)
- new net GPIO3: MCU1.11 (PA4)
- new net GPIO4: MCU1.12 (PA5)
- new net HEARTBEAT: MCU1.13 (PA6), R6.1
- new net HighChan1: C3.2, MCU1.30 (PB6), R3.1
- new net HighChan2: C4.2, MCU1.31 (PB7), R4.1
- new net HighChan3: C5.2, R5.1
- new net LowChan1: C1.2, MCU1.27 (PB3), R1.1
- new net LowChan2: C2.2, MCU1.28 (PB4), R2.1
- new net LowChan3: MCU1.29 (PB5)
- new net NRST: MCU1.6 (PF2)
- new net SWCLK: MCU1.25 (PA14)
- new net SWDIO: MCU1.24 (PA13)
- new net WKUP: MCU1.7 (PA0)
- no-connect marks 0 -> 9
Other:
- note added: "- LowChan and HighChan are gpio outputs, controlling the low and high current load drivers respectively - All MCU pins are connected via buses, which connect to other hierarchical sheets - GPIO[0..4] are to be used as needed later. Connector is TBD. The first 3 are capable of GPIO or PWM output. - Channel buttons (used for debugging) are connected with RC low pass filter for button debouncing. Ti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"
- note added: "Channel Buttons (for debugging)"
- note added: "Design Notes"
- note added: "Global/Hierarchical Labels"
- note added: "Labels and LEDs"
- note added: "STM32G0B1"
