File: Hardware/STM32G0B1.kicad_sch (KiCad schematic)
At the start: 36 parts, among them SW1 SW_Push, SW2 SW_Push, SW3 SW_Push, SW4 SW_Push, SW5 SW_Push, SW6 SW_Push, SW7 SW_Push, SW8 SW_Push, Y1 Crystal

Commit message: temp
Connections:
- net Chan1: now also C2.2, R2.1; no longer C3.2, R3.1
- net Chan2: now also C3.2, R3.1; no longer C5.2, R5.1
- net Chan3: now also C4.2, R4.1; no longer C7.2, R7.1
- net Chan4: now also C5.2, R5.1; no longer C2.2, R2.1
- net Chan5: now also C6.2, R6.1; no longer C4.2, R4.1
- net Chan6: now also C7.2, R7.1; no longer C6.2, R6.1
Changed lines of the file:
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@@
 	)
 	(label "Chan5"
-		(at 256.54 58.42 180)
+		(at 256.54 76.2 180)
 		(effects
 			(font
@@
 	)
 	(label "Chan3"
-		(at 194.31 93.98 180)
+		(at 256.54 58.42 180)
 		(effects
 			(font
@@
 	)
 	(label "Chan4"
-		(at 256.54 40.64 180)
+		(at 194.31 76.2 180)
 		(effects
 			(font
@@
 	)
 	(label "Chan1"
-		(at 194.31 58.42 180)
+		(at 256.54 40.64 180)
 		(effects
 			(font
@@
 	)
 	(label "Chan2"
-		(at 194.31 76.2 180)
+		(at 194.31 58.42 180)
 		(effects
 			(font
@@
 	)
 	(label "Chan6"
-		(at 256.54 76.2 180)
-		(effects
-			(font
+		(at 194.31 93.98 180)
+		(effects
+			(font
