File: Hardware/old.kicad_sch (KiCad schematic)
At the start: 52 parts, among them J1 DT13-2P, J2 Conn_01x04_Pin, J3 Conn_01x03_Pin, U1 STM32G0B1KETx, U2 AP63203WU-7, U3 AP63205WU-7, U4 ISOW1044, U5 TPS4H160AQPWPRQ1

Commit message: Finished the STM sheet mostly
- Added a bus for the STM32, as well as the individual peripherals
- Added LEDs for the Heartbeat and Fault outputs.
- Added 5 pushbuttons for the 5 channels, along with button debouncing
	- Refer to TI's button debouncing AN. RC low pass w/ 10ms time
	  constant. UNSURE if the schematic is correct, someone will
	  have to check.
Parts:
- removed U1: STM32G0B1KETx, Package_QFP:LQFP-32_7x7mm_P0.8mm, symbol MCU_ST_STM32G0:STM32G0B1KETx
Changed lines of the file:
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@@
-	)
-	(symbol
-		(lib_id "MCU_ST_STM32G0:STM32G0B1KETx")
-		(at 144.78 195.58 0)
-		(unit 1)
-		(exclude_from_sim no)
-		(in_bom yes)
-		(on_board yes)
-		(dnp no)
-		(property "Reference" "U1"
-			(at 146.9233 165.1 0)
-			(effects
-				(font
-					(size 1.27 1.27)
-				)
-				(justify left)
-			)
-		)
-		(property "Value" "STM32G0B1KETx"
-			(at 146.9233 167.64 0)
-			(effects
-				(font
-					(size 1.27 1.27)
-				)
-				(justify left)
-			)
-		)
-		(property "Footprint" "Package_QFP:LQFP-32_7x7mm_P0.8mm"
-			(at 121.92 218.44 0)
-			(effects
-				(font
-					(size 1.27 1.27)
-				)
-				(justify right)
-				(hide yes)
-			)
-		)
-		(property "Datasheet" "https://www.st.com/resource/en/datasheet/stm32g0b1ke.pdf"
-			(at 144.78 195.58 0)
-			(effects
-				(font
-					(size 1.27 1.27)
-				)
-				(hide yes)
-			)
-		)
-		(property "Description" "STMicroelectronics Arm Cortex-M0+ MCU, 512KB flash, 144KB RAM, 64 MHz, 1.7-3.6V, 30 GPIO, LQFP32"
-			(at 144.78 195.58 0)
-			(effects
-				(font
-					(size 1.27 1.27)
-				)
-				(hide yes)
-			)
-		)
-		(pin "6"
-		)
-		(pin "20"
-		)
-		(pin "2"
-		)
-		(pin "3"
-		)
-		(pin "15"
-		)
-		(pin "18"
-		)
-		(pin "10"
-		)
-		(pin "31"
-		)
-		(pin "16"
-		)
-		(pin "12"
-		)
-		(pin "7"
-		)
-		(pin "28"
-		)
-		(pin "30"
-		)
-		(pin "13"
-		)
-		(pin "14"
-		)
-		(pin "23"
-		)
-		(pin "24"
-		)
-		(pin "29"
-		)
-		(pin "32"
-		)
-		(pin "22"
-		)
-		(pin "25"
-		)
-		(pin "27"
-		)
-		(pin "5"
-		)
-		(pin "17"
-		)
-		(pin "21"
-		)
-		(pin "1"
-		)
-		(pin "11"
-		)
-		(pin "4"
-		)
-		(pin "8"
-		)
-		(pin "19"
-		)
-		(pin "9"
-		)
-		(pin "26"
-		)
-		(instances
-			(project "CANIO-Board"
-				(path "/a11f98b2-3b09-4cf9-8535-19e509fe91b9/fc1f1a73-316b-40ab-bfc3-5dfc259e0898"
-					(reference "U1")
-					(unit 1)
-				)
-			)
-		)
 	)
 	(symbol
