File: Hardware/Power.kicad_sch (KiCad schematic)
At the start: 0 parts

Commit message: Added the power schematic
- Finished the power schematic.
- HOWEVER, there is some confusion (Arnav) about the post-supply
  filtering. Needs to be reviewed before ordering.

Co-authored-by: Nicholas Nunez <ngnunez@icloud.com>
Parts:
- added BUCK1: AP63203WU, Package_TO_SOT_SMD:TSOT-23-6, symbol Regulator_Switching:AP63203WU
- added BUCK2: AP63205WU, Package_TO_SOT_SMD:TSOT-23-6, symbol Regulator_Switching:AP63205WU
- added C10, C6: 10u, symbol Device:C_Small_US
- added C11, C7: 100n, symbol Device:C_Small_US
- added C12, C13, C8, C9: 22u, symbol Device:C_Small_US
- added L1, L2: 4.7u, symbol Device:L_Small
Connections:
- new net: BUCK2.5 (SW), C11.1, L2.1
- new net: BUCK1.5 (SW), C7.1, L1.1
- new net: BUCK1.6 (BST), C7.2
- new net: BUCK2.6 (BST), C11.2
- new net +12V: BUCK1.2 (EN), BUCK1.3 (IN), BUCK2.2 (EN), BUCK2.3 (IN), C10.1, C6.1
- new net 3v3: BUCK1.1 (FB), C8.1, C9.1, L1.2
- new net 5v0: BUCK2.1 (FB), C12.1, C13.1, L2.2
- new net GND: BUCK1.4 (GND), BUCK2.4 (GND), C10.2, C12.2, C13.2, C6.2, C8.2, C9.2
Other:
- note added: "- All parts of the schematic are from the manufacturer's datasheet. - HOWEVER: What is currently UNCLEAR is the 4.7uH and 2x22uF filtering setup at the output of each IC. Needs to be reviewed. - Illustration at https://www.desmos.com/calculator/au2a0t2rlf"
- note added: "Buck Converters"
- note added: "Design Notes"
