File: Hardware/Power.kicad_sch (KiCad schematic)
At the start: 17 parts

Commit message: temp
Parts:
- added DT1: Conn_01x02, footprints:TE_DTF13-2P, symbol Connector_Generic:Conn_01x02
- added SCREW1: Conn_01x02, TerminalBlock:TerminalBlock_MaiXu_MX126-5.0-02P_1x02_P5.00mm, symbol Connector_Generic:Conn_01x02
Connections:
- net +12V: now also DT1.1 (Pin_1), SCREW1.1 (Pin_1)
- net GND: now also DT1.2 (Pin_2), SCREW1.2 (Pin_2)
