File: Hardware/Connectors.kicad_sch (KiCad schematic)
At the start: 24 parts, among them J3 Conn_01x05, J4 TC2030, J5 Conn_01x03, J6 USB_C_Receptacle_USB2.0_14P, SW6 SW_Push, SW7 SW_Push

Commit message: Fixed up the schematic a little, and did *most* footprint assigning
- Most footprints are assigned. Ones that arent either don't exist, or
  are out of stock at digikey and are thus not work making/adding.
- Details of next steps will be put into changelog soon
Parts:
- removed J3: Conn_01x05, symbol Connector_Generic:Conn_01x05
- removed WAGO1, WAGO2: 2606, symbol Connector_Generic:Conn_01x02
- removed WAGO3, WAGO4, WAGO5: 2601, symbol Connector_Generic:Conn_01x02
- added J1: Conn_01x07, Connector_PinHeader_2.54mm:PinHeader_1x07_P2.54mm_Vertical, symbol Connector_Generic:Conn_01x07
- added R18: 10k, Resistor_SMD:R_0603_1608Metric_Pad0.98x0.95mm_HandSolder, symbol Device:R_Small_US
- added WAGO1: 2606, symbol Connector_Generic:Conn_01x04
- added WAGO2: 2601, TerminalBlock_WAGO:TerminalBlock_WAGO_2601-1106_1x06_P3.50mm_Horizontal, symbol Connector_Generic:Conn_01x06
- C28: renamed from C20; footprint (none) -> Capacitor_SMD:C_0603_1608Metric_Pad1.08x0.95mm_HandSolder
- C29: renamed from C21; footprint (none) -> Capacitor_SMD:C_0603_1608Metric_Pad1.08x0.95mm_HandSolder
- DIP1: footprint (none) -> Button_Switch_THT:SW_DIP_SPSTx03_Slide_9.78x9.8mm_W7.62mm_P2.54mm
- DT1: renamed from TD1; footprint (none) -> TerminalBlock:TerminalBlock_MaiXu_MX126-5.0-02P_1x02_P5.00mm
- FILTER2: renamed from FILTER1; value ECMF2-40A100N6 -> ECMF02-2AMX6
- J2: renamed from J5; footprint (none) -> Connector_PinHeader_2.54mm:PinHeader_1x03_P2.54mm_Vertical
- R13: renamed from R15; footprint (none) -> Resistor_SMD:R_0603_1608Metric_Pad0.98x0.95mm_HandSolder
- R14: renamed from R16; value 20k -> 10k; footprint (none) -> Resistor_SMD:R_0603_1608Metric_Pad0.98x0.95mm_HandSolder
- R15: renamed from R17; footprint (none) -> Resistor_SMD:R_0603_1608Metric_Pad0.98x0.95mm_HandSolder
- R16: renamed from R13; footprint (none) -> Resistor_SMD:R_0603_1608Metric_Pad0.98x0.95mm_HandSolder
- R17: renamed from R14; footprint (none) -> Resistor_SMD:R_0603_1608Metric_Pad0.98x0.95mm_HandSolder
- SW6, SW7: footprint (none) -> Button_Switch_SMD:SW_Push_1P1T_NO_CK_KSC7xxJ
- TVS3, TVS4, TVS5: footprint (none) -> Package_TO_SOT_SMD:SOT-23-5
- renumbered J4 to TC1, J6 to USB1
Connections:
- net GND: now also R18.2, WAGO1.2 (Pin_2), WAGO1.4 (Pin_4), WAGO2.2 (Pin_2), WAGO2.4 (Pin_4), WAGO2.6 (Pin_6); no longer R14.2
- net GPIO0: now also J1.1 (Pin_1)
- net GPIO1: now also J1.2 (Pin_2)
- net GPIO2: now also J1.3 (Pin_3)
- net GPIO3: now also J1.4 (Pin_4)
- net GPIO4: now also J1.5 (Pin_5)
- net HighDriveOut1: now also WAGO1.1 (Pin_1)
- net HighDriveOut2: now also WAGO1.3 (Pin_3)
- net LowDrive1: now also WAGO2.1 (Pin_1)
- net LowDrive2: now also WAGO2.3 (Pin_3)
- net LowDrive3: now also WAGO2.5 (Pin_5)
- net GPIO6: now reaches TVS3.3 (IN2)
- net GPIO6: now also J1.7 (Pin_7)
- net GPIO5: now reaches TVS3.4 (IN3)
- net GPIO5: now also J1.6 (Pin_6)
- new net: R14.2, R18.1
- no-connect marks 5 -> 3
Other:
- moved on the sheet: R14, TVS3, TVS4
