File: Hardware/Connectors.kicad_sch (KiCad schematic)
At the start: 23 parts, among them J1 Conn_01x03, J2 Conn_01x07, SW9 SW_Push

Commit message: temp
Parts:
- added H1, H2, H3, H4: GND, MountingHole:MountingHole_3.5mm_Pad_Via, symbol Mechanical:MountingHole_Pad
- DT1: footprint (none) -> TerminalBlock:TerminalBlock_MaiXu_MX126-5.0-03P_1x03_P5.00mm
- FILTER2: footprint (none) -> footprints:ECMF02-2AMX6_QFN-6L
- USB1: footprint (none) -> footprints:SHOUHAN_TYPE-C_16PIN_2MD__073_
- WAGO1, WAGO2, WAGO3, WAGO4, WAGO5, WAGO6, WAGO7, WAGO8: footprint (none) -> TerminalBlock_WAGO:TerminalBlock_WAGO_2601-1102_1x02_P3.50mm_Horizontal
Connections:
- net GND: now also H1.1, H2.1, H3.1, H4.1
Other:
- note added: "Reset and Mounting Holes"
- note removed: "Reset"

Commit message: temp
Parts:
- added SCREW2: Conn_01x03, TerminalBlock:TerminalBlock_MaiXu_MX126-5.0-03P_1x03_P5.00mm, symbol Connector_Generic:Conn_01x03
- DT2: renamed from DT1; footprint TerminalBlock:TerminalBlock_MaiXu_MX126-5.0-03P_1x03_P5.00mm -> footprints:TE_DTF13-3P
Connections:
- net CANH_+: now also SCREW2.1 (Pin_1)
- net CANL_-: now also SCREW2.2 (Pin_2)
- net GND: now also SCREW2.3 (Pin_3); no longer WAGO1.2 (Pin_2), WAGO2.2 (Pin_2), WAGO3.2 (Pin_2), WAGO4.2 (Pin_2), WAGO5.2 (Pin_2), WAGO6.2 (Pin_2), WAGO7.2 (Pin_2), WAGO8.2 (Pin_2)
- net DriverOut0 renamed DriverOutP0
- net DriverOut1 renamed DriverOutP1
- net DriverOut2 renamed DriverOutP2
- net DriverOut3 renamed DriverOutP3
- net DriverOut4 renamed DriverOutP4
- net DriverOut5 renamed DriverOutP5
- net DriverOut6 renamed DriverOutP6
- net DriverOut7 renamed DriverOutP7
- new net DriverOutN0: WAGO1.2 (Pin_2)
- new net DriverOutN1: WAGO2.2 (Pin_2)
- new net DriverOutN2: WAGO3.2 (Pin_2)
- new net DriverOutN3: WAGO4.2 (Pin_2)
- new net DriverOutN4: WAGO5.2 (Pin_2)
- new net DriverOutN5: WAGO6.2 (Pin_2)
- new net DriverOutN6: WAGO7.2 (Pin_2)
- new net DriverOutN7: WAGO8.2 (Pin_2)
Other:
- moved on the sheet: DT2
