File: Hardware/CANIO-Board.kicad_pcb (KiCad board)
At the start: 4 copper layers, 0 parts

Commit message: temp
Parts:
- added BUCK1: AP63203QWU-7, Package_TO_SOT_SMD:TSOT-23-6, F.Cu at (193.8, 95.7)
- added BUCK2: AP63205QWU-7, Package_TO_SOT_SMD:TSOT-23-6, F.Cu at (421.0, 106.0)
- added C1: 1u, Capacitor_SMD:C_0603_1608Metric_Pad1.08x0.95mm_HandSolder, F.Cu at (130.0, 117.0)
- added C10: 100n, Capacitor_SMD:C_0603_1608Metric_Pad1.08x0.95mm_HandSolder, F.Cu at (369.3, 93.5)
- added C11: 10u, Capacitor_SMD:C_0603_1608Metric_Pad1.08x0.95mm_HandSolder, F.Cu at (369.3, 96.0)
- added C12: 100n, Capacitor_SMD:C_0603_1608Metric_Pad1.08x0.95mm_HandSolder, F.Cu at (369.3, 98.5)
- added C13: 22n, Capacitor_SMD:C_0603_1608Metric_Pad1.08x0.95mm_HandSolder, F.Cu at (373.6, 86.0)
- added C14: 22n, Capacitor_SMD:C_0603_1608Metric_Pad1.08x0.95mm_HandSolder, F.Cu at (373.6, 88.5)
- added C15: 100n, Capacitor_SMD:C_0603_1608Metric_Pad1.08x0.95mm_HandSolder, F.Cu at (197.8, 95.7)
- added C16: 22u, Capacitor_SMD:CP_Elec_4x4.5, F.Cu at (184.5, 101.2)
- added C17: 22u, Capacitor_SMD:CP_Elec_4x4.5, F.Cu at (184.5, 95.3)
- added C18: 10u, Capacitor_SMD:C_0603_1608Metric_Pad1.08x0.95mm_HandSolder, F.Cu at (189.8, 95.7)
- added C19: 100n, Capacitor_SMD:C_0603_1608Metric_Pad1.08x0.95mm_HandSolder, F.Cu at (416.3, 91.0)
- added C2: 1u, Capacitor_SMD:C_0603_1608Metric_Pad1.08x0.95mm_HandSolder, F.Cu at (142.2, 117.0)
- added C20: 22u, Capacitor_SMD:CP_Elec_4x4.5, F.Cu at (410.2, 99.4)
- added C21: 22u, Capacitor_SMD:CP_Elec_4x4.5, F.Cu at (410.2, 105.2)
- added C22: 10u, Capacitor_SMD:C_0603_1608Metric_Pad1.08x0.95mm_HandSolder, F.Cu at (416.3, 93.5)
- added C23: 10u, Capacitor_SMD:C_0603_1608Metric_Pad1.08x0.95mm_HandSolder, F.Cu at (384.4, 86.0)
- added C24: 10u, Capacitor_SMD:C_0603_1608Metric_Pad1.08x0.95mm_HandSolder, F.Cu at (384.4, 88.5)
- added C25: 4.7u, Capacitor_SMD:C_0603_1608Metric_Pad1.08x0.95mm_HandSolder, F.Cu at (384.4, 91.0)
- added C26: 10n, Capacitor_SMD:C_0603_1608Metric_Pad1.08x0.95mm_HandSolder, F.Cu at (384.4, 93.5)
- added C27: 1u, Capacitor_SMD:C_0603_1608Metric_Pad1.08x0.95mm_HandSolder, F.Cu at (375.3, 57.5)
- added C3: 1u, Capacitor_SMD:C_0603_1608Metric_Pad1.08x0.95mm_HandSolder, F.Cu at (170.0, 117.0)
- added C4: 1u, Capacitor_SMD:C_0603_1608Metric_Pad1.08x0.95mm_HandSolder, F.Cu at (182.2, 117.0)
- added C5: 1u, Capacitor_SMD:C_0603_1608Metric_Pad1.08x0.95mm_HandSolder, F.Cu at (130.0, 129.0)
- added C6: 1u, Capacitor_SMD:C_0603_1608Metric_Pad1.08x0.95mm_HandSolder, F.Cu at (142.1, 127.1)
- added C7: 1u, Capacitor_SMD:C_0603_1608Metric_Pad1.08x0.95mm_HandSolder, F.Cu at (170.0, 129.0)
- added C8: 1u, Capacitor_SMD:C_0603_1608Metric_Pad1.08x0.95mm_HandSolder, F.Cu at (182.2, 129.0)
- added C9: 10u, Capacitor_SMD:C_0603_1608Metric_Pad1.08x0.95mm_HandSolder, F.Cu at (369.3, 91.0)
- added CAN1: ISO1042, Package_SO:SOIC-16W_7.5x10.3mm_P1.27mm, F.Cu at (393.0, 90.8)
- added DCDC1: NME1, footprints:NME1S, F.Cu at (393.3, 100.6)
- added DIP1: SW_DIP_x03, Button_Switch_THT:SW_DIP_SPSTx03_Slide_9.78x9.8mm_W7.62mm_P2.54mm, F.Cu at (113.5, 117.3)
- added DT1: Conn_01x03, TerminalBlock:TerminalBlock_MaiXu_MX126-5.0-03P_1x03_P5.00mm, F.Cu at (359.6, 53.6)
- added FILTER1: ECMF02-2AMX6, footprints:ECMF02-2AMX6_QFN-6L, F.Cu at (401.2, 91.2)
- added FILTER2: ECMF02-2AMX6, footprints:ECMF02-2AMX6_QFN-6L, F.Cu at (150.0, 125.0)
- added H1: GND, MountingHole:MountingHole_3.5mm_Pad_Via, F.Cu at (104.2, 90.0)
- added H2: GND, MountingHole:MountingHole_3.5mm_Pad_Via, F.Cu at (195.8, 90.0)
- added H3: GND, MountingHole:MountingHole_3.5mm_Pad_Via, F.Cu at (195.8, 130.8)
- added H4: GND, MountingHole:MountingHole_3.5mm_Pad_Via, F.Cu at (104.2, 130.8)
- added J1: Conn_01x03, Connector_PinHeader_2.54mm:PinHeader_1x03_P2.54mm_Vertical, F.Cu at (379.8, 58.6)
- added J2: Conn_01x07, Connector_PinHeader_2.54mm:PinHeader_1x07_P2.54mm_Vertical, F.Cu at (185.4, 116.5)
- added L1: 4.7u, Inductor_THT:L_Axial_L7.0mm_D3.3mm_P5.08mm_Vertical_Fastron_MICC, F.Cu at (195.8, 100.7)
- added L2: 4.7u, Inductor_THT:L_Axial_L7.0mm_D3.3mm_P5.08mm_Vertical_Fastron_MICC, F.Cu at (420.9, 96.6)
- added L3: 47u, Inductor_THT:L_Axial_L7.0mm_D3.3mm_P5.08mm_Vertical_Fastron_MICC, F.Cu at (388.9, 107.1)
- added LDO1: SPX5205-ADJ, Package_TO_SOT_SMD:SOT-23-5_HandSoldering, F.Cu at (398.5, 107.1)
- added LED1: LED_Small, LED_SMD:LED_1206_3216Metric_Pad1.42x1.75mm_HandSolder, F.Cu at (377.2, 101.5)
- added LED2: LED_Small, LED_SMD:LED_1206_3216Metric_Pad1.42x1.75mm_HandSolder, F.Cu at (377.2, 104.9)
- added LED3: LED_Small, LED_SMD:LED_1206_3216Metric_Pad1.42x1.75mm_HandSolder, F.Cu at (426.6, 100.7)
- added LED4: LED_Small, LED_SMD:LED_1206_3216Metric_Pad1.42x1.75mm_HandSolder, F.Cu at (426.6, 104.1)
- added MCU1: STM32G0B1KETxN, Package_QFP:LQFP-32_7x7mm_P0.8mm, F.Cu at (150.0, 115.0)
- added R1: 10k, Resistor_SMD:R_0603_1608Metric_Pad0.98x0.95mm_HandSolder, F.Cu at (117.8, 113.0)
- added R10: 1k, Resistor_SMD:R_0603_1608Metric_Pad0.98x0.95mm_HandSolder, F.Cu at (378.0, 98.5)
- added R11: 1k, Resistor_SMD:R_0603_1608Metric_Pad0.98x0.95mm_HandSolder, F.Cu at (416.3, 96.0)
- added R12: 1k, Resistor_SMD:R_0603_1608Metric_Pad0.98x0.95mm_HandSolder, F.Cu at (416.3, 98.5)
- added R13: 17k, Resistor_SMD:R_0603_1608Metric_Pad0.98x0.95mm_HandSolder, F.Cu at (384.4, 96.0)
- added R14: 10k, Resistor_SMD:R_0603_1608Metric_Pad0.98x0.95mm_HandSolder, F.Cu at (384.4, 98.5)
- added R15: 10k, Resistor_SMD:R_0603_1608Metric_Pad0.98x0.95mm_HandSolder, F.Cu at (384.4, 101.0)
- added R16: 10k, Resistor_SMD:R_0603_1608Metric_Pad0.98x0.95mm_HandSolder, F.Cu at (384.4, 103.6)
- added R17: 5.1k, Resistor_SMD:R_0603_1608Metric_Pad0.98x0.95mm_HandSolder, F.Cu at (142.5, 131.2)
- added R18: 5.1k, Resistor_SMD:R_0603_1608Metric_Pad0.98x0.95mm_HandSolder, F.Cu at (157.5, 131.2)
- added R19: 10k, Resistor_SMD:R_0603_1608Metric_Pad0.98x0.95mm_HandSolder, F.Cu at (375.3, 65.1)
- added R2: 10k, Resistor_SMD:R_0603_1608Metric_Pad0.98x0.95mm_HandSolder, F.Cu at (130.0, 113.0)
- added R3: 10k, Resistor_SMD:R_0603_1608Metric_Pad0.98x0.95mm_HandSolder, F.Cu at (157.8, 113.0)
- added R4: 10k, Resistor_SMD:R_0603_1608Metric_Pad0.98x0.95mm_HandSolder, F.Cu at (170.0, 113.0)
- added R5: 10k, Resistor_SMD:R_0603_1608Metric_Pad0.98x0.95mm_HandSolder, F.Cu at (117.8, 125.0)
- added R6: 10k, Resistor_SMD:R_0603_1608Metric_Pad0.98x0.95mm_HandSolder, F.Cu at (130.0, 125.0)
- added R7: 10k, Resistor_SMD:R_0603_1608Metric_Pad0.98x0.95mm_HandSolder, F.Cu at (157.8, 125.0)
- added R8: 10k, Resistor_SMD:R_0603_1608Metric_Pad0.98x0.95mm_HandSolder, F.Cu at (170.0, 125.0)
- added R9: 1k, Resistor_SMD:R_0603_1608Metric_Pad0.98x0.95mm_HandSolder, F.Cu at (378.0, 96.0)
- added SW1: SW_Push, Button_Switch_SMD:SW_Push_1P1T_NO_CK_KSC7xxJ, F.Cu at (123.9, 115.0)
- added SW2: SW_Push, Button_Switch_SMD:SW_Push_1P1T_NO_CK_KSC7xxJ, F.Cu at (136.1, 115.0)
- added SW3: SW_Push, Button_Switch_SMD:SW_Push_1P1T_NO_CK_KSC7xxJ, F.Cu at (163.9, 115.0)
- added SW4: SW_Push, Button_Switch_SMD:SW_Push_1P1T_NO_CK_KSC7xxJ, F.Cu at (176.1, 115.0)
- added SW5: SW_Push, Button_Switch_SMD:SW_Push_1P1T_NO_CK_KSC7xxJ, F.Cu at (123.9, 127.0)
- added SW6: SW_Push, Button_Switch_SMD:SW_Push_1P1T_NO_CK_KSC7xxJ, F.Cu at (136.1, 127.0)
- added SW7: SW_Push, Button_Switch_SMD:SW_Push_1P1T_NO_CK_KSC7xxJ, F.Cu at (163.9, 127.0)
- added SW8: SW_Push, Button_Switch_SMD:SW_Push_1P1T_NO_CK_KSC7xxJ, F.Cu at (176.1, 127.0)
- added SW9: SW_Push, Button_Switch_SMD:SW_Push_1P1T_NO_CK_KSC7xxJ, F.Cu at (378.2, 52.4)
- added TC1: TC2030, Connector:Tag-Connect_TC2030-IDC-NL_2x03_P1.27mm_Vertical, F.Cu at (377.2, 68.8)
- added TVS1: D_TVS, Diode_SMD:D_SMA_Handsoldering, F.Cu at (423.5, 87.0)
- added TVS2: D_TVS_Dual_AAC, Package_TO_SOT_SMD:SOT-23, F.Cu at (401.9, 87.1)
- added TVS3: ESDS314DBVR, Package_TO_SOT_SMD:SOT-23-5, F.Cu at (358.2, 61.0)
- added TVS4: ESDS314DBVR, Package_TO_SOT_SMD:SOT-23-5, F.Cu at (358.2, 65.7)
- added TVS5: ESDS314DBVR, Package_TO_SOT_SMD:SOT-23-5, F.Cu at (358.2, 70.3)
- added USB1: USB_C_Receptacle_USB2.0_16P, footprints:SHOUHAN_TYPE-C_16PIN_2MD__073_, F.Cu at (150.0, 132.2)
- added WAGO1: 2601, TerminalBlock_WAGO:TerminalBlock_WAGO_2601-1102_1x02_P3.50mm_Horizontal, F.Cu at (109.5, 73.2)
- added WAGO2: 2601, TerminalBlock_WAGO:TerminalBlock_WAGO_2601-1102_1x02_P3.50mm_Horizontal, F.Cu at (121.6, 73.2)
- added WAGO3: 2601, TerminalBlock_WAGO:TerminalBlock_WAGO_2601-1102_1x02_P3.50mm_Horizontal, F.Cu at (133.7, 73.2)
- added WAGO4: 2601, TerminalBlock_WAGO:TerminalBlock_WAGO_2601-1102_1x02_P3.50mm_Horizontal, F.Cu at (145.8, 73.2)
- added WAGO5: 2601, TerminalBlock_WAGO:TerminalBlock_WAGO_2601-1102_1x02_P3.50mm_Horizontal, F.Cu at (157.9, 73.2)
- added WAGO6: 2601, TerminalBlock_WAGO:TerminalBlock_WAGO_2601-1102_1x02_P3.50mm_Horizontal, F.Cu at (170.0, 73.2)
- added WAGO7: 2601, TerminalBlock_WAGO:TerminalBlock_WAGO_2601-1102_1x02_P3.50mm_Horizontal, F.Cu at (182.1, 73.2)
- added WAGO8: 2601, TerminalBlock_WAGO:TerminalBlock_WAGO_2601-1102_1x02_P3.50mm_Horizontal, F.Cu at (194.2, 73.2)
- added Y1: Crystal, Crystal:Crystal_SMD_3215-2Pin_3.2x1.5mm, F.Cu at (376.7, 108.2)
Routing:
- added copper zone on B.Cu, net +12V
- added copper zone on F.Cu, net GND
- added copper zone on In1.Cu, net GND
Other:
- board outline added: 100 x 70 mm
- board text added: "- Board is centered at (150, 100), and is 100mm*70mm. - Corners have 3mm fillet. PTHs are 3.5mm (support M3 screws) - Bottom PTHs are 4.25mm away from both edges. Top ones are 4.25mm away from the left and right edges, and 25mm away from the top edge. These are all from edge of board to center of PTH. - MCU is 15mm below the center of the board, tilted 45 degrees for optimal routing. - Allocated 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"
- board text added: "3v3"
- board text added: "Design Notes"
- board text added: "GPIO6"
- board text added: "Layer 1 - GND"
- board text added: "Layer 2 - GND"
- board text added: "Layer 4 - 12V"
- board text added: "PB6"
- board text added: "PB7"
- board text added: "PB9 - GPIO0"
- board text added: "PD0"
- board text added: "PD1"
- board text added: "PD2"
- board text added: "PD3"
- board text added: "RESERVED for Load Driver"

Commit message: temp
Parts:
- moved CAN1 284.1 mm to (110.1, 117.7), turned to 180 degrees
- moved DCDC1 283.2 mm to (110.1, 101.0), turned to 180 degrees
- moved BUCK2 227.4 mm to (193.6, 110.8)
- moved C22 227.3 mm to (189.6, 110.8), turned to 90 degrees
- moved C20 226.2 mm to (184.6, 116.1), turned to 180 degrees
- moved L2 226.1 mm to (195.6, 115.8), turned to 180 degrees
- moved C21 225.7 mm to (184.6, 110.3), turned to 180 degrees
- moved C19 219.5 mm to (197.6, 110.8), turned to 90 degrees
- moved C6 10.0 mm to (142.1, 137.1)
- moved C1 10.0 mm to (130.0, 127.0)
- moved C2 10.0 mm to (142.2, 127.0)
- moved C3 10.0 mm to (170.0, 127.0)
- moved C4 10.0 mm to (182.2, 127.0)
- moved C5 10.0 mm to (130.0, 139.0)
- moved C7 10.0 mm to (170.0, 139.0)
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Routing:
- added copper zone on F.Cu, net CANGND
- added copper zone on B.Cu, net CANVDD
Other:
- board size 100 x 70 mm -> 100 x 80 mm
- board text added: "- Board is centered at (150, 100), and is 100mm*80mm. - Corners have 3mm fillet. PTHs are 3.5mm (support M3 screws) - Bottom PTHs are 4.25mm away from both edges. Top ones are 4.25mm away from the left and right edges, and 25mm away from the top edge. These are all from edge of board to center of PTH. - MCU is 20mm below the center of the board, tilted 45 degrees for optimal routing. - Allocated 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"
- board text added: "5v0"
- board text added: "Load Driver"
- board text added: "NO Copper Pour on In1 under CANH/L1!! Also, CANGND and CANVDD on top and bottom"
- board text removed: "- Board is centered at (150, 100), and is 100mm*70mm. - Corners have 3mm fillet. PTHs are 3.5mm (support M3 screws) - Bottom PTHs are 4.25mm away from both edges. Top ones are 4.25mm away from the left and right edges, and 25mm away from the top edge. These are all from edge of board to center of PTH. - MCU is 15mm below the center of the board, tilted 45 degrees for optimal routing. - Allocated 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"

Commit message: temp
Parts:
- added DFB1: D_Small, Diode_THT:D_DO-35_SOD27_P7.62mm_Horizontal, F.Cu at (125.8, 109.5)
- added DFB2: D_Small, Diode_THT:D_DO-35_SOD27_P7.62mm_Horizontal, F.Cu at (133.4, 112.0)
- added DFB3: D_Small, Diode_THT:D_DO-35_SOD27_P7.62mm_Horizontal, F.Cu at (141.5, 109.5)
- added DFB4: D_Small, Diode_THT:D_DO-35_SOD27_P7.62mm_Horizontal, F.Cu at (149.2, 112.0)
- added DFB5: D_Small, Diode_THT:D_DO-35_SOD27_P7.62mm_Horizontal, F.Cu at (157.2, 109.5)
- added DFB6: D_Small, Diode_THT:D_DO-35_SOD27_P7.62mm_Horizontal, F.Cu at (165.0, 112.0)
- added DFB7: D_Small, Diode_THT:D_DO-35_SOD27_P7.62mm_Horizontal, F.Cu at (172.9, 109.5)
- added DFB8: D_Small, Diode_THT:D_DO-35_SOD27_P7.62mm_Horizontal, F.Cu at (179.9, 112.0)
- added DT1: Conn_01x02, footprints:TE_DTF13-2P, F.Cu at (186.3, 132.5)
- added LOAD1: TBD62783AFWG, Package_SO:SOP-18_7x12.5mm_P1.27mm, F.Cu at (169.1, 119.5)
- added RELAY1: ALDP112W, footprints:RELAY_ALDP112W, F.Cu at (121.9, 95.8)
- added RELAY2: ALDP112W, footprints:RELAY_ALDP112W, F.Cu at (129.8, 95.8)
- added RELAY3: ALDP112W, footprints:RELAY_ALDP112W, F.Cu at (137.6, 95.8)
- added RELAY4: ALDP112W, footprints:RELAY_ALDP112W, F.Cu at (145.4, 95.8)
- added RELAY5: ALDP112W, footprints:RELAY_ALDP112W, F.Cu at (153.2, 95.8)
- added RELAY6: ALDP112W, footprints:RELAY_ALDP112W, F.Cu at (161.0, 95.8)
- added RELAY7: ALDP112W, footprints:RELAY_ALDP112W, F.Cu at (168.9, 95.8)
- added RELAY8: ALDP112W, footprints:RELAY_ALDP112W, F.Cu at (176.7, 95.8)
- added SB1: SolderJumper_2_Open, Jumper:SolderJumper-2_P1.3mm_Open_TrianglePad1.0x1.5mm, F.Cu at (122.0, 117.0)
- added SB10: SolderJumper_2_Open, Jumper:SolderJumper-2_P1.3mm_Open_TrianglePad1.0x1.5mm, F.Cu at (127.0, 120.0)
- added SB11: SolderJumper_2_Open, Jumper:SolderJumper-2_P1.3mm_Open_TrianglePad1.0x1.5mm, F.Cu at (131.9, 120.0)
- added SB12: SolderJumper_2_Open, Jumper:SolderJumper-2_P1.3mm_Open_TrianglePad1.0x1.5mm, F.Cu at (136.9, 120.0)
- added SB13: SolderJumper_2_Open, Jumper:SolderJumper-2_P1.3mm_Open_TrianglePad1.0x1.5mm, F.Cu at (141.9, 117.0)
- added SB14: SolderJumper_2_Open, Jumper:SolderJumper-2_P1.3mm_Open_TrianglePad1.0x1.5mm, F.Cu at (146.9, 117.0)
- added SB15: SolderJumper_2_Open, Jumper:SolderJumper-2_P1.3mm_Open_TrianglePad1.0x1.5mm, F.Cu at (151.9, 117.0)
- added SB16: SolderJumper_2_Open, Jumper:SolderJumper-2_P1.3mm_Open_TrianglePad1.0x1.5mm, F.Cu at (156.9, 117.0)
- added SB17: SolderJumper_2_Open, Jumper:SolderJumper-2_P1.3mm_Open_TrianglePad1.0x1.5mm, F.Cu at (141.9, 123.0)
- added SB18: SolderJumper_2_Open, Jumper:SolderJumper-2_P1.3mm_Open_TrianglePad1.0x1.5mm, F.Cu at (146.9, 123.0)
- added SB19: SolderJumper_2_Open, Jumper:SolderJumper-2_P1.3mm_Open_TrianglePad1.0x1.5mm, F.Cu at (151.9, 123.0)
- added SB2: SolderJumper_2_Open, Jumper:SolderJumper-2_P1.3mm_Open_TrianglePad1.0x1.5mm, F.Cu at (127.0, 117.0)
- added SB20: SolderJumper_2_Open, Jumper:SolderJumper-2_P1.3mm_Open_TrianglePad1.0x1.5mm, F.Cu at (156.9, 123.0)
- added SB21: SolderJumper_2_Open, Jumper:SolderJumper-2_P1.3mm_Open_TrianglePad1.0x1.5mm, F.Cu at (141.9, 120.0)
- added SB22: SolderJumper_2_Open, Jumper:SolderJumper-2_P1.3mm_Open_TrianglePad1.0x1.5mm, F.Cu at (146.9, 120.0)
- added SB23: SolderJumper_2_Open, Jumper:SolderJumper-2_P1.3mm_Open_TrianglePad1.0x1.5mm, F.Cu at (151.9, 120.0)
- added SB24: SolderJumper_2_Open, Jumper:SolderJumper-2_P1.3mm_Open_TrianglePad1.0x1.5mm, F.Cu at (156.9, 120.0)
- added SB3: SolderJumper_2_Open, Jumper:SolderJumper-2_P1.3mm_Open_TrianglePad1.0x1.5mm, F.Cu at (131.9, 117.0)
- added SB4: SolderJumper_2_Open, Jumper:SolderJumper-2_P1.3mm_Open_TrianglePad1.0x1.5mm, F.Cu at (136.9, 117.0)
- added SB5: SolderJumper_2_Open, Jumper:SolderJumper-2_P1.3mm_Open_TrianglePad1.0x1.5mm, F.Cu at (122.0, 123.0)
- added SB6: SolderJumper_2_Open, Jumper:SolderJumper-2_P1.3mm_Open_TrianglePad1.0x1.5mm, F.Cu at (127.0, 123.0)
- added SB7: SolderJumper_2_Open, Jumper:SolderJumper-2_P1.3mm_Open_TrianglePad1.0x1.5mm, F.Cu at (131.9, 123.0)
- added SB8: SolderJumper_2_Open, Jumper:SolderJumper-2_P1.3mm_Open_TrianglePad1.0x1.5mm, F.Cu at (136.9, 123.0)
- added SB9: SolderJumper_2_Open, Jumper:SolderJumper-2_P1.3mm_Open_TrianglePad1.0x1.5mm, F.Cu at (122.0, 120.0)
- added SCREW1: Conn_01x02, TerminalBlock:TerminalBlock_MaiXu_MX126-5.0-02P_1x02_P5.00mm, F.Cu at (171.2, 134.0)
- added SCREW2: Conn_01x03, TerminalBlock:TerminalBlock_MaiXu_MX126-5.0-03P_1x03_P5.00mm, F.Cu at (106.9, 136.3)
- DT2: renamed from DT1; footprint TerminalBlock:TerminalBlock_MaiXu_MX126-5.0-03P_1x03_P5.00mm -> footprints:TE_DTF13-3P
- moved FILTER1 298.2 mm to (104.3, 119.3), turned to 90 degrees
- moved DT2 259.5 mm to (112.2, 131.8), turned to -90 degrees
- moved C1 20.0 mm to (130.0, 147.0)
- moved C2 20.0 mm to (142.2, 147.0)
- moved C3 20.0 mm to (170.0, 147.0)
- moved C4 20.0 mm to (182.2, 147.0)
- moved C5 20.0 mm to (130.0, 159.0)
- moved C6 20.0 mm to (142.1, 157.1)
- moved C7 20.0 mm to (170.0, 159.0)
- moved C8 20.0 mm to (182.2, 159.0)
- moved DIP1 20.0 mm to (113.5, 147.3)
- moved FILTER2 20.0 mm to (150.0, 155.0)
- moved H3 20.0 mm to (195.8, 160.8)
- moved H4 20.0 mm to (104.2, 160.8)
- moved J2 20.0 mm to (185.4, 146.5)
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Connections:
- WAGO1 pad 1: /Connectors/DriverOut0 -> /Connectors/DriverOutP0
- WAGO1 pad 2: GND -> /Connectors/DriverOutN0
- WAGO2 pad 1: /Connectors/DriverOut1 -> /Connectors/DriverOutP1
- WAGO2 pad 2: GND -> /Connectors/DriverOutN1
- WAGO3 pad 1: /Connectors/DriverOut2 -> /Connectors/DriverOutP2
- WAGO3 pad 2: GND -> /Connectors/DriverOutN2
- WAGO4 pad 1: /Connectors/DriverOut3 -> /Connectors/DriverOutP3
- WAGO4 pad 2: GND -> /Connectors/DriverOutN3
- WAGO5 pad 1: /Connectors/DriverOut4 -> /Connectors/DriverOutP4
- WAGO5 pad 2: GND -> /Connectors/DriverOutN4
- WAGO6 pad 1: /Connectors/DriverOut5 -> /Connectors/DriverOutP5
- WAGO6 pad 2: GND -> /Connectors/DriverOutN5
- WAGO7 pad 1: /Connectors/DriverOut6 -> /Connectors/DriverOutP6
- WAGO7 pad 2: GND -> /Connectors/DriverOutN6
- WAGO8 pad 1: /Connectors/DriverOut7 -> /Connectors/DriverOutP7
- WAGO8 pad 2: GND -> /Connectors/DriverOutN7
Routing:
- net /Connectors/DriverOutN7: track 0.00 -> 74.4 mm, vias 0 -> 1
- net /Connectors/DriverOutN6: track 0.00 -> 66.9 mm, vias 0 -> 2
- net /Connectors/DriverOutN5: track 0.00 -> 63.2 mm, vias 0 -> 2
- net /Connectors/DriverOutN4: track 0.00 -> 61.6 mm, vias 0 -> 2
- net Net-(SB16-B): track 0.00 -> 60.0 mm, vias 0 -> 2
- net /Connectors/DriverOutN2: track 0.00 -> 58.9 mm, vias 0 -> 2
- net /Connectors/DriverOutN1: track 0.00 -> 57.6 mm, vias 0 -> 2
- net /Connectors/DriverOutN3: track 0.00 -> 57.2 mm, vias 0 -> 2
- net /Connectors/DriverOutN0: track 0.00 -> 55.1 mm, vias 0 -> 1
- net +12V: track 0.00 -> 54.8 mm, vias 0 -> 17
- net /Load_Driver/Coil0: track 0.00 -> 53.9 mm, vias 0 -> 2
- net Net-(SB15-B): track 0.00 -> 51.4 mm, vias 0 -> 2
- net Net-(SB14-B): track 0.00 -> 49.4 mm, vias 0 -> 3
- net Net-(SB4-B): track 0.00 -> 47.1 mm, vias 0 -> 2
- net Net-(SB13-B): track 0.00 -> 47.0 mm, vias 0 -> 3
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Other:
- board size 100 x 80 mm -> 100 x 100 mm
- board text added: "- Board is centered at (150, 115), and is 100mm*100mm. - Corners have 3mm fillet. PTHs are 3.5mm (support M3 screws) - Bottom PTHs are 4.25mm away from both edges. Top ones are 4.25mm away from the left and right edges, and 25mm away from the top edge. These are all from edge of board to center of PTH. - MCU is 20mm below the center of the board, tilted 45 degrees for optimal routing. - Allocated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"
- board text added: "This entire area does not use 3v3 or 5v0. In2 can be used to route signals."
- board text removed: "- Board is centered at (150, 100), and is 100mm*80mm. - Corners have 3mm fillet. PTHs are 3.5mm (support M3 screws) - Bottom PTHs are 4.25mm away from both edges. Top ones are 4.25mm away from the left and right edges, and 25mm away from the top edge. These are all from edge of board to center of PTH. - MCU is 20mm below the center of the board, tilted 45 degrees for optimal routing. - Allocated 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"
- board text removed: "RESERVED for Load Driver"
