File: Hardware/Load_Driver.kicad_sch (KiCad schematic)
At the start: 0 parts

Commit message: temp
Parts:
- added PLACEHOLDER1: Conn_01x08, symbol Connector_Generic:Conn_01x08
Connections:
- new net DriverOut0: PLACEHOLDER1.1 (Pin_1)
- new net DriverOut1: PLACEHOLDER1.2 (Pin_2)
- new net DriverOut2: PLACEHOLDER1.3 (Pin_3)
- new net DriverOut3: PLACEHOLDER1.4 (Pin_4)
- new net DriverOut4: PLACEHOLDER1.5 (Pin_5)
- new net DriverOut5: PLACEHOLDER1.6 (Pin_6)
- new net DriverOut6: PLACEHOLDER1.7 (Pin_7)
- new net DriverOut7: PLACEHOLDER1.8 (Pin_8)
Other:
- note added: "Placeholder! Delete and replace with Load Driver"

Commit message: temp
Parts:
- removed PLACEHOLDER1: Conn_01x08, symbol Connector_Generic:Conn_01x08
- added DFB1, DFB2, DFB3, DFB4, DFB5, DFB6, DFB7, DFB8: D_Small, Diode_THT:D_DO-35_SOD27_P7.62mm_Horizontal, symbol Device:D_Small
- added F1, F2, F3, F4, F5, F6, F7, F8: 5A, Fuse:Fuseholder_Blade_Mini_Keystone_3568, symbol Device:Fuse
- added LOAD1: TBD62783AFWG, Package_SO:SOP-18_7x12.5mm_P1.27mm, symbol symbols:TBD62783AFWG
- added RELAY1, RELAY2, RELAY3, RELAY4, RELAY5, RELAY6, RELAY7, RELAY8: J1071CS12VDC.36, Relay_THT:Relay_SPDT_Finder_36.11, symbol Relay:FINDER-36.11
- added SB1, SB10, SB11, SB12, SB13, SB14, SB15, SB16, SB17, SB18, SB19, SB2, SB20, SB21, SB22, SB23, SB24, SB3, SB4, SB5, SB6, SB7, SB8, SB9: SolderJumper_2_Open, footprints:SolderBridge, symbol Jumper:SolderJumper_2_Open
Connections:
- new net: RELAY8.11, SB19.1 (A), SB20.2 (B)
- new net: F6.1, RELAY6.14
- new net: RELAY3.11, SB5.1 (A), SB6.2 (B)
- new net: RELAY2.11, SB3.1 (A), SB4.2 (B)
- new net: F2.1, RELAY2.14
- new net: RELAY6.11, SB15.1 (A), SB16.2 (B)
- new net: RELAY1.11, SB1.1 (A), SB2.2 (B)
- new net: F1.1, RELAY1.14
- new net: RELAY4.11, SB7.1 (A), SB8.2 (B)
- new net: RELAY5.11, SB13.1 (A), SB14.2 (B)
- new net: F5.1, RELAY5.14
- new net: F3.1, RELAY3.14
- new net: RELAY7.11, SB17.1 (A), SB18.2 (B)
- new net: F4.1, RELAY4.14
- new net: F7.1, RELAY7.14
- new net: F8.1, RELAY8.14
- new net +12V: LOAD1.9 (VCC), SB1.2 (B), SB13.2 (B), SB15.2 (B), SB17.2 (B), SB19.2 (B), SB3.2 (B), SB5.2 (B), SB7.2 (B)
- new net Chan0: LOAD1.1 (IN1)
- new net Chan1: LOAD1.2 (IN2)
- new net Chan2: LOAD1.3 (IN3)
- new net Chan3: LOAD1.4 (IN4)
- new net Chan4: LOAD1.5 (IN5)
- new net Chan5: LOAD1.6 (IN6)
- new net Chan6: LOAD1.7 (IN7)
- new net Chan7: LOAD1.8 (IN8)
- new net Coil0: DFB1.1 (K), LOAD1.18 (OUT1), RELAY1.A1
- new net Coil1: DFB2.1 (K), LOAD1.17 (OUT2), RELAY2.A1
- new net Coil2: DFB3.1 (K), LOAD1.16 (OUT3), RELAY3.A1
- new net Coil3: DFB4.1 (K), LOAD1.15 (OUT4), RELAY4.A1
- new net Coil4: DFB5.1 (K), LOAD1.14 (OUT5), RELAY5.A1
- new net Coil5: DFB6.1 (K), LOAD1.13 (OUT6), RELAY6.A1
- new net Coil6: DFB7.1 (K), LOAD1.12 (OUT7), RELAY7.A1
- new net Coil7: DFB8.1 (K), LOAD1.11 (OUT8), RELAY8.A1
- new net DriverOutN0: SB2.1 (A), SB9.1 (A)
- new net DriverOutN1: SB10.1 (A), SB4.1 (A)
- new net DriverOutN2: SB11.1 (A), SB6.1 (A)
- new net DriverOutN3: SB12.1 (A), SB8.1 (A)
- new net DriverOutN4: SB14.1 (A), SB21.1 (A)
- new net DriverOutN5: SB16.1 (A), SB22.1 (A)
- new net DriverOutN6: SB18.1 (A), SB23.1 (A)
- new net DriverOutN7: SB20.1 (A), SB24.1 (A)
- new net DriverOutP0: F1.2
- new net DriverOutP1: F2.2
- new net DriverOutP2: F3.2
- new net DriverOutP3: F4.2
- new net DriverOutP4: F5.2
- new net DriverOutP5: F6.2
- new net DriverOutP6: F7.2
- new net DriverOutP7: F8.2
- new net GND: DFB1.2 (A), DFB2.2 (A), DFB3.2 (A), DFB4.2 (A), DFB5.2 (A), DFB6.2 (A), DFB7.2 (A), DFB8.2 (A), LOAD1.10 (GND), RELAY1.A2, RELAY2.A2, RELAY3.A2, RELAY4.A2, RELAY5.A2, RELAY6.A2, RELAY7.A2, RELAY8.A2, SB10.2 (B), SB11.2 (B), SB12.2 (B), SB21.2 (B), SB22.2 (B), SB23.2 (B), SB24.2 (B), SB9.2 (B)
- no-connect marks 0 -> 8
Other:
- note added: "- The load driver IC is an 8 channel high side switch, that can supply upto 500mA per channel with Vcc upto 50V. - The high side switch is used to power 8 relay coils, which each draw 12V 30mA (0.36W). The relays themselves are capable of supplying upto 15A constant. - The solder bridges allow you to select from the WAGO connector output being 12V-GND, or just a connected/disconnected wire. - For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"
- note added: "Load Driver High Side Switch and Relays"
- note removed: "- The load driver ICs are the recommended TPL7407LA's. - The drivers themselves have only 7 channels, from which we need 2 and have to double up on 3 more. - Thus, to split the current evenly (put equal load on both ICs), I've set one HighDrive (single channel running a relay coil) per IC, and an additional doubled up LowDrive (1.6A direct draw) per IC. Then, for the last LowDrive, I've split it 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"
- note removed: "Placeholder! Delete and replace with Load Driver"

Commit message: temp
Parts:
- removed F1, F2, F3, F4, F5, F6, F7, F8: 5A, Fuse:Fuseholder_Blade_Mini_Keystone_3568, symbol Device:Fuse
- removed RELAY1, RELAY2, RELAY3, RELAY4, RELAY5, RELAY6, RELAY7, RELAY8: J1071CS12VDC.36, Relay_THT:Relay_SPDT_Finder_36.11, symbol Relay:FINDER-36.11
- added RELAY1, RELAY2, RELAY3, RELAY4, RELAY5, RELAY6, RELAY7, RELAY8: ALDP112W, footprints:RELAY_ALDP112W, symbol symbols:ALDP112W
- SB1, SB10, SB11, SB12, SB13, SB14, SB15, SB16, SB17, SB18, SB19, SB2, SB20, SB21, SB22, SB23, SB24, SB3, SB4, SB5, SB6, SB7, SB8, SB9: footprint footprints:SolderBridge -> Jumper:SolderJumper-2_P1.3mm_Open_TrianglePad1.0x1.5mm
Connections:
- net +12V: now also SB1.1 (A), SB13.1 (A), SB14.1 (A), SB15.1 (A), SB16.1 (A), SB2.1 (A), SB3.1 (A), SB4.1 (A); no longer SB1.2 (B), SB13.2 (B), SB15.2 (B), SB17.2 (B), SB19.2 (B), SB3.2 (B), SB5.2 (B), SB7.2 (B)
- net Coil0: now also RELAY1.1
- net Coil1: now also RELAY2.1
- net Coil2: now also RELAY3.1
- net Coil3: now also RELAY4.1
- net Coil4: now also RELAY5.1
- net Coil5: now also RELAY6.1
- net Coil6: now also RELAY7.1
- net Coil7: now also RELAY8.1
- net DriverOutN0: now also SB5.2 (B); no longer SB2.1 (A)
- net DriverOutN1: now also SB6.2 (B); no longer SB4.1 (A)
- net DriverOutN2: now also SB7.2 (B); no longer SB6.1 (A)
- net DriverOutN3: now also SB8.2 (B); no longer SB8.1 (A)
- net DriverOutN4: now also SB17.2 (B); no longer SB14.1 (A)
- net DriverOutN5: now also SB18.2 (B); no longer SB16.1 (A)
- net DriverOutN6: now also SB19.2 (B); no longer SB18.1 (A)
- net DriverOutN7: now also SB20.2 (B); no longer SB20.1 (A)
- net DriverOutP0: now also RELAY1.3
- net DriverOutP1: now also RELAY2.3
- net DriverOutP2: now also RELAY3.3
- net DriverOutP3: now also RELAY4.3
- net DriverOutP4: now also RELAY5.3
- net DriverOutP5: now also RELAY6.3
- net DriverOutP6: now also RELAY7.3
- net DriverOutP7: now also RELAY8.3
- net GND: now also RELAY1.2, RELAY2.2, RELAY3.2, RELAY4.2, RELAY5.2, RELAY6.2, RELAY7.2, RELAY8.2
- net at SB19.1 (A): now also SB15.2 (B), RELAY7.4; no longer SB20.2 (B)
- net at SB5.1 (A): now also SB1.2 (B), RELAY1.4; no longer SB6.2 (B)
- net at SB4.2 (B): now also SB8.1 (A), RELAY4.4; no longer SB3.1 (A)
- net at SB16.2 (B): now also SB20.1 (A), RELAY8.4; no longer SB15.1 (A)
- net at SB2.2 (B): now also SB6.1 (A), RELAY2.4; no longer SB1.1 (A)
- net at SB7.1 (A): now also SB3.2 (B), RELAY3.4; no longer SB8.2 (B)
- net at SB14.2 (B): now also SB18.1 (A), RELAY6.4; no longer SB13.1 (A)
- net at SB17.1 (A): now also SB13.2 (B), RELAY5.4; no longer SB18.2 (B)
- no-connect marks 8 -> 0
Other:
- moved on the sheet: DFB1, LOAD1, SB1
